File: pcb/submission.kicad_pcb (KiCad board)
At the start: 2 copper layers, 198.4 x 84.1 mm, 109 parts, among them J1 USB_C_Receptacle_USB2.0, SW0 RotaryEncoder_Switch, SW1 RotaryEncoder_Switch, U1 STM32F072CBT6, U2 PRTR5V0U2X, U3 XC6206PxxxMR-Regulator_Linear

Commit message: Updated pcb silkscreen
Other:
- board text added: "submission 1.0.1 (2024)"
- board text removed: "submission 1.0 (2024) github.com/mhzkb"
